Commit message: Made changes to mjcf for inertia, controller debugs

File: mjcf/robot/turtlebot3_burger.urdf (robot description, URDF)
Before this commit: robot turtlebot3_burger, 7 links, 6 joints
Links:
- link base_link: geometry visual mesh filename=burger_base.stl scale=0.001 0.001 0.001
- link base_scan: geometry visual mesh filename=lds.stl scale=0.001 0.001 0.001
- link wheel_left_link: geometry visual mesh filename=left_tire.stl scale=0.001 0.001 0.001
- link wheel_right_link: geometry visual mesh filename=right_tire.stl scale=0.001 0.001 0.001
